File: KiCad/H_Bridge_BLDC/H_Bridge_BLDC.kicad_pcb (KiCad board)
At the start: 2 copper layers, 100 x 200 mm, 131 parts, among them J1 DriveCoil, J10 Conn_02x15_Counter_Clockwise, J2 HallDec, J3 Ctrl, J4 12V, J5 Hall In, J6 Hall Out, J7 Conn_02x15_Counter_Clockwise, J8 Conn_02x15_Counter_Clockwise, J9 Conn_02x15_Counter_Clockwise, Q1 2N5401, Q10 2N5551, Q11 2N5551, Q12 2N5551, Q13 2N5551, Q14 2N5551, Q15 2N5551, Q16 2N5551, Q17 2N5551, Q18 2N5401, Q2 BDW94C, Q3 BDW93C, Q4 BDW93C, Q5 BDW94C, Q6 2N5401, Q7 2N5401, Q8 2N5401, Q9 2N5551, U1 VO615A, U2 L7805CV, U3 CD74HC238E, U4 VO615A, U6 LM555xM, U7 LM555xM

Commit message: Added BOM and changed some parts (same footprint)
Parts:
- C1, C7: value 470uF -> 470uF 63V
- C3, C4, C5, C6: value 470uF 250V -> 470uF 63V
- FL1: value SU9V-07010 -> SU9VF-07015
Changed lines of the file:
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@@
 		(tags "Through hole pin header THT 1x05 2.54mm single row")
 		(property "Reference" "J5"
-			(at 0 -2.33 360)
+			(at 0 -2.33 0)
 			(layer "F.SilkS")
 			(effects
@@
 		)
 		(property "Value" "Hall In"
-			(at 0 12.49 360)
+			(at 0 12.49 0)
 			(layer "F.Fab")
 			(effects
@@
 		(tags "to-92 sc-43 sc-43a sot54 PA33 transistor")
 		(property "Reference" "Q8"
-			(at -1.7 -3.12 360)
+			(at -1.7 -3.12 0)
 			(layer "F.SilkS")
 			(effects
@@
 		)
 		(property "Value" "2N5401"
-			(at 1.27 2.79 360)
+			(at 1.27 2.79 0)
 			(layer "F.Fab")
 			(effects
@@
 		)
 		(fp_text user "${REFERENCE}"
-			(at 1.27 0 360)
+			(at 1.27 0 0)
 			(layer "F.Fab")
 			(effects
@@
 		(tags "to-92 sc-43 sc-43a sot54 PA33 transistor")
 		(property "Reference" "Q16"
-			(at -1.9 -3.2 360)
+			(at -1.9 -3.2 0)
 			(layer "F.SilkS")
 			(effects
@@
 		)
 		(property "Value" "2N5551"
-			(at 1 4 360)
+			(at 1 4 0)
 			(layer "F.Fab")
 			(effects
@@
 		)
 		(fp_text user "${REFERENCE}"
-			(at 1.27 0 360)
+			(at 1.27 0 0)
 			(layer "F.Fab")
 			(effects
@@
 			)
 		)
-		(property "Value" "470uF"
+		(property "Value" "470uF 63V"
 			(at -1.939823 6 90)
 			(layer "F.Fab")
@@
 			)
 		)
-		(property "Datasheet" ""
+		(property "Datasheet" "https://search.kemet.com/download/datasheet/ESK477M063AL4EA"
 			(at 0 0 90)
 			(unlocked yes)
@@
 		(tags "to-92 sc-43 sc-43a sot54 PA33 transistor")
 		(property "Reference" "Q14"
-			(at -2 -3.2 360)
+			(at -2 -3.2 0)
 			(layer "F.SilkS")
 			(effects
@@
 		)
 		(property "Value" "2N5551"
-			(at 1 4.5 360)
+			(at 1 4.5 0)
 			(layer "F.Fab")
 			(effects
@@
 		)
 		(fp_text user "${REFERENCE}"
-			(at 1.27 0 360)
+			(at 1.27 0 0)
 			(layer "F.Fab")
 			(effects
@@
 			)
 		)
-		(property "Value" "SU9V-07010"
+		(property "Value" "SU9VF-07015"
 			(at -10.5 0 90)
 			(layer "F.Fab")
@@
 			)
 		)
-		(property "Description" "1 mH @ 1 kHz 2 Lijn Common Mode Choke Through-hole 700mA DCR 600mOhm"
+		(property "Description" "1.5 mH @ 1 kHz 2 Common Mode Choke Through-hole 700mA"
 			(at 0 0 0)
 			(layer "F.Fab")
@@
 			)
 		)
-		(property "Digikey" "https://www.digikey.nl/short/fbcjc4v0"
+		(property "Digikey" "https://www.digikey.nl/short/8qzt38p9"
 			(at 0 0 180)
 			(unlocked yes)
@@
 		(tags "to-92 sc-43 sc-43a sot54 PA33 transistor")
 		(property "Reference" "Q13"
-			(at -1.9 -3.12 360)
+			(at -1.9 -3.12 0)
 			(layer "F.SilkS")
 			(effects
@@
 		)
 		(property "Value" "2N5551"
-			(at 1.27 2.79 360)
+			(at 1.27 2.79 0)
 			(layer "F.Fab")
 			(effects
@@
 		)
 		(fp_text user "${REFERENCE}"
-			(at 1.27 0 360)
+			(at 1.27 0 0)
 			(layer "F.Fab")
 			(effects
@@
 			)
 		)
-		(property "Value" "470uF 250V"
+		(property "Value" "470uF 63V"
 			(at 2.5 6.25 0)
 			(layer "F.Fab")
@@
 			)
 		)
-		(property "Datasheet" "https://mm.digikey.com/Volume0/opasdata/d220001/medias/docus/2452/ECA-xxM%20Series%2CTypeA.pdf"
+		(property "Datasheet" "https://search.kemet.com/download/datasheet/ESK477M063AL4EA"
 			(at 0 0 180)
 			(unlocked yes)
@@
 			)
 		)
-		(property "Digikey" "https://www.digikey.nl/short/nq94djb8"
+		(property "Digikey" "https://www.digikey.nl/short/2thtjq03"
 			(at 0 0 180)
 			(unlocked yes)
@@
 		(tags "to-92 sc-43 sc-43a sot54 PA33 transistor")
 		(property "Reference" "Q15"
-			(at -1.8 -3.1 360)
+			(at -1.8 -3.1 0)
 			(layer "F.SilkS")
 			(effects
@@
 		)
 		(property "Value" "2N5551"
-			(at 1.27 2.79 360)
+			(at 1.27 2.79 0)
 			(layer "F.Fab")
 			(effects
@@
 		)
 		(fp_text user "${REFERENCE}"
-			(at 1.27 0 360)
+			(at 1.27 0 0)
 			(layer "F.Fab")
 			(effects
@@
 			)
 		)
-		(property "Value" "470uF"
+		(property "Value" "470uF 63V"
 			(at -3.5 3.25 90)
 			(layer "F.Fab")
@@
 			)
 		)
-		(property "Datasheet" ""
+		(property "Datasheet" "https://search.kemet.com/download/datasheet/ESK477M063AL4EA"
 			(at 0 0 0)
 			(unlocked yes)
@@
 		(tags "to-92 sc-43 sc-43a sot54 PA33 transistor")
 		(property "Reference" "Q18"
-			(at -2 -3 360)
+			(at -2 -3 0)
 			(layer "F.SilkS")
 			(effects
@@
 		)
 		(property "Value" "2N5401"
-			(at 1.27 2.79 360)
+			(at 1.27 2.79 0)
 			(layer "F.Fab")
 			(effects
@@
 		)
 		(fp_text user "${REFERENCE}"
-			(at 1.27 0 360)
+			(at 1.27 0 0)
 			(layer "F.Fab")
 			(effects
@@
 		(tags "to-92 sc-43 sc-43a sot54 PA33 transistor")
 		(property "Reference" "Q17"
-			(at -2 -3.2 360)
+			(at -2 -3.2 0)
 			(layer "F.SilkS")
 			(effects
@@
 		)
 		(property "Value" "2N5551"
-			(at 1.27 2.79 360)
+			(at 1.27 2.79 0)
 			(layer "F.Fab")
 			(effects
@@
 		)
 		(fp_text user "${REFERENCE}"
-			(at 1.27 0 360)
+			(at 1.27 0 0)
 			(layer "F.Fab")
 			(effects
@@
 		(tags "to-92 sc-43 sc-43a sot54 PA33 transistor")
 		(property "Reference" "Q12"
-			(at -2.4 -3.2 360)
+			(at -2.4 -3.2 0)
 			(layer "F.SilkS")
 			(effects
@@
 		)
 		(property "Value" "2N5551"
-			(at 1 4.5 360)
+			(at 1 4.5 0)
 			(layer "F.Fab")
 			(effects
@@
 		)
 		(fp_text user "${REFERENCE}"
-			(at 1.27 0 360)
+			(at 1.27 0 0)
 			(layer "F.Fab")
 			(effects
@@
 		(tags "to-92 sc-43 sc-43a sot54 PA33 transistor")
 		(property "Reference" "Q10"
-			(at 1.27 -3.56 360)
+			(at 1.27 -3.56 0)
 			(layer "F.SilkS")
 			(effects
@@
 		)
 		(property "Value" "2N5551"
-			(at 1.27 2.79 360)
+			(at 1.27 2.79 0)
 			(layer "F.Fab")
 			(effects
@@
 		)
 		(fp_text user "${REFERENCE}"
-			(at 1.27 0 360)
+			(at 1.27 0 0)
 			(layer "F.Fab")
 			(effects
@@
 			)
 		)
-		(property "Value" "470uF 250V"
+		(property "Value" "470uF 63V"
 			(at 2.5 6.25 0)
 			(layer "F.Fab")
@@
 			)
 		)
-		(property "Datasheet" "https://mm.digikey.com/Volume0/opasdata/d220001/medias/docus/2452/ECA-xxM%20Series%2CTypeA.pdf"
+		(property "Datasheet" "https://search.kemet.com/download/datasheet/ESK477M063AL4EA"
 			(at 0 0 180)
 			(unlocked yes)
@@
 			)
 		)
-		(property "Digikey" "https://www.digikey.nl/short/nq94djb8"
+		(property "Digikey" "https://www.digikey.nl/short/2thtjq03"
 			(at 0 0 180)
 			(unlocked yes)
@@
 		)
 		(fp_text user "${REFERENCE}"
-			(at 0 2.54 360)
+			(at 0 2.54 0)
 			(layer "F.Fab")
 			(effects
@@
 			)
 		)
-		(property "Value" "470uF 250V"
+		(property "Value" "470uF 63V"
 			(at 2.5 6.25 0)
 			(layer "F.Fab")
@@
 			)
 		)
-		(property "Datasheet" "https://mm.digikey.com/Volume0/opasdata/d220001/medias/docus/2452/ECA-xxM%20Series%2CTypeA.pdf"
+		(property "Datasheet" "https://search.kemet.com/download/datasheet/ESK477M063AL4EA"
 			(at 0 0 180)
 			(unlocked yes)
@@
 			)
 		)
-		(property "Digikey" "https://www.digikey.nl/short/nq94djb8"
+		(property "Digikey" "https://www.digikey.nl/short/2thtjq03"
 			(at 0 0 180)
 			(unlocked yes)
@@
 		(tags "to-92 sc-43 sc-43a sot54 PA33 transistor")
 		(property "Reference" "Q7"
-			(at -1.4 -3.2 360)
+			(at -1.4 -3.2 0)
 			(layer "F.SilkS")
 			(effects
@@
 		)
 		(property "Value" "2N5401"
-			(at 1.27 2.79 360)
+			(at 1.27 2.79 0)
 			(layer "F.Fab")
 			(effects
@@
 		)
 		(fp_text user "${REFERENCE}"
-			(at 1.27 0 360)
+			(at 1.27 0 0)
 			(layer "F.Fab")
 			(effects
@@
 			)
 		)
-		(property "Value" "470uF 250V"
+		(property "Value" "470uF 63V"
 			(at 2.5 6.25 0)
 			(layer "F.Fab")
@@
 			)
 		)
-		(property "Datasheet" "https://mm.digikey.com/Volume0/opasdata/d220001/medias/docus/2452/ECA-xxM%20Series%2CTypeA.pdf"
+		(property "Datasheet" "https://search.kemet.com/download/datasheet/ESK477M063AL4EA"
 			(at 0 0 180)
 			(unlocked yes)
@@
 			)
 		)
-		(property "Digikey" "https://www.digikey.nl/short/nq94djb8"
+		(property "Digikey" "https://www.digikey.nl/short/2thtjq03"
 			(at 0 0 180)
 			(unlocked yes)
@@
 		(tags "TO-220-3 Vertical RM 2.54mm")
 		(property "Reference" "U2"
-			(at -3.9225 -0.80625 180)
+			(at -3.9225 -0.80625 0)
 			(layer "F.SilkS")
 			(effects
@@
 			)
 		)
-		(property "DigiKey" "https://www.digikey.nl/short/7nprw4r0"
+		(property "Digikey" "https://www.digikey.nl/short/7nprw4r0"
 			(at 0 0 -90)
 			(unlocked yes)
